File: kicad/powermatic_1200/powermatic_1200.kicad_pcb (KiCad board)
At the start: 2 copper layers, 461.5 x 461.5 mm, 64 parts, among them J1 T4171310004-001, K1 HMC-9B30-11-DS, K2 HC3096N-52-900-24, K3 HMC-9B30-11-DS, K4 HMC-9B30-11-DS, K5 HMC-9B30-11-DS, K6 HMC-9B30-11-DS, Q1 FAZ-D4/2-NA-L, SW1 222102

Commit message: Update enclosure BOM, footprint artwork, and assembly model alignment
Preserve detailed drawings on F.Fab, use simplified F.SilkS outlines and F.Adhes fills, and align contactor accessories to the nominal Fusion assembly. Include current schematic and terminal placement edits, model verification tools, and review artifacts.

Record reconciliation with the shared parts rail export. KiCad loads all 58 board footprints, model checks pass, and the schematic netlist exports successfully. Nominal assembly alignment is not a collision-free fit approval.
Parts:
- removed the REF** at (19.3, 22.7)
- removed the REF** at (40.0, 442.0)
- removed the REF** at (20.0, 441.0)
- removed the REF** at (41.0, 231.8)
- removed the REF** at (4.60, 533.6)
- removed the TB23 at (176.0, 319.4)
- moved TB12 311.2 mm to (236.0, 216.3)
- moved TB14 311.2 mm to (241.0, 216.3)
- moved TB16 311.2 mm to (246.0, 216.3)
- moved MI1 304.3 mm to (395.4, 361.0)
- moved TB10 301.2 mm to (221.0, 216.3)
- moved TB2 301.2 mm to (201.0, 216.3)
- moved TB4 301.2 mm to (206.0, 216.3)
- moved TB6 301.2 mm to (211.0, 216.3)
- moved TB8 301.2 mm to (216.0, 216.3)
- moved SP2 223.7 mm to (340.8, 337.4)
- moved K3 223.5 mm to (340.8, 369.4)
- moved TB18 201.8 mm to (360.0, 263.6)
- moved TB20 201.8 mm to (365.0, 263.6)
- moved TB21 201.8 mm to (350.0, 263.6)
- moved TB23 201.8 mm to (355.0, 263.6)
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