File: kicad/powermatic_1200/powermatic_1200.kicad_pcb (KiCad board)
At the start: 24 copper layers, 462 x 716 mm, 157 parts, among them J1 T4171310004-001, J2 3PH-4W-PLUG, J3 BSPBX-22-W, J4 BSPDX-23-W, J5 Frame_PE_Lug_20mm, J6 J6, J7 Frame_PE_Lug_20mm, K1 HMC-9B30-11-DS, K2 HMC-9B30-11-DS, K3 HC3096N-52-900-24, K4 HMC-9B30-11-DS, K5 HMC-9B30-11-DS, K6 HMC-9B30-11-DS, M1 PWRM1200-MOTOR, Q1 FAZ-D4/2-NA-L, SW1 222102

Commit message: Bond all DIN rails and refresh wire schedule
Parts:
- added TB98: KN-G12SP-10, Controls:KN-G12SP-10_Front, F.Cu at (391.0, 67.0)
- moved REF** 6.00 mm to (401.0, 67.0)
Routing:
- net PE: track 5953.8 -> 6206.1 mm
