File: kicad/powermatic_1200/powermatic_1200.kicad_pcb (KiCad board)
At the start: 24 copper layers, 462 x 716 mm, 159 parts, among them J1 T4171310004-001, J2 3PH-4W-PLUG, J3 BSPBX-22-W, J4 BSPDX-23-W, J5 Frame_PE_Lug_20mm, J6 J6, J7 Frame_PE_Lug_20mm, J8 Frame_PE_Lug_20mm, K1 HMC-9B30-11-DS, K2 HMC-9B30-11-DS, K3 HC3096N-52-900-24, K4 HMC-9B30-11-DS, K5 HMC-9B30-11-DS, K6 HMC-9B30-11-DS, M1 PWRM1200-MOTOR, Q1 FAZ-D4/2-NA-L, SW1 222102

Commit message: Use supplied door bond and separate J-box grounding branches
Parts:
- moved J8 19.3 mm to (449.3, 449.3)
Routing:
- net PE: track 6713.1 -> 6723.7 mm
Changed lines of the file:
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@@
 			)
 		)
-		(property "Wire.BondingPlan" "TB50.1 to J8.PE lower-right enclosure/backplate grounding stud: 12 AWG green/yellow, 10 mm single ferrule at TB50.1 and McMaster 9388K35 5/16 in ring at J8. Routed; retain the four backplate mounting/bonding interfaces."
+		(property "Wire.BondingPlan" "TB50.1 to J8.PE: 12 AWG green/yellow to the existing lower-right enclosure grounding fixture on User.Drawings; endpoint concentric at (449.2876,449.2876) mm. 10 mm single ferrule at TB50.1; owner-selected 5/16 in McMaster 9388K35 ring at the lug."
 			(at 0 0 0)
 			(layer "F.Fab")
@@
 			)
 		)
-		(property "Wire.SuppliedBond" "{\"schema\":1,\"sku\":\"GRDKIT01\",\"supplier\":\"Hammond\",\"wire\":\"existing_frame_PE\",\"awg\":10,\"supplied_length_mm\":304.8,\"termination_at_lug\":\"factory ring retained\",\"status\":\"routed\",\"from\":\"J7.PE motor bell stud\",\"to\":\"J5.PE drill press frame\",\"termination_at_motor_stud\":\"factory ring retained\"}"
+		(property "Wire.SuppliedBond" "{\"schema\":1,\"sku\":\"GRDKIT01\",\"supplier\":\"Hammond\",\"wire\":\"existing_frame_PE\",\"awg\":10,\"supplied_length_mm\":304.8,\"termination_at_lug\":\"factory ring retained\",\"status\":\"routed\",\"from\":\"M1.PE motor-box WAGO 221-613 splice\",\"to\":\"J5.PE drill press frame\",\"termination_at_splice\":\"ring removed; bare copper, 13 mm strip\"}"
 			(at 343 749 0)
 			(layer "F.Fab")
@@
 			)
 		)
-		(property "Wire.SplicePlan.PE" "{\"schema\":1,\"connector\":\"WAGO 221-613\",\"ports\":[{\"wire\":\"motor_PE_to_gland\",\"awg\":12,\"strip_mm\":13},{\"wire\":\"motor-body-bond\",\"to\":\"J7.PE\",\"awg\":10,\"strip_mm\":13,\"status\":\"routed\"},{\"status\":\"unused\"}]}"
+		(property "Wire.SplicePlan.PE" "{\"schema\":1,\"connector\":\"WAGO 221-613\",\"ports\":[{\"wire\":\"motor_PE_to_gland\",\"awg\":12,\"strip_mm\":13},{\"wire\":\"motor-body-bond\",\"to\":\"J7.PE\",\"awg\":10,\"strip_mm\":13,\"status\":\"routed\"},{\"wire\":\"machine-frame-bond\",\"to\":\"J5.PE\",\"awg\":10,\"strip_mm\":13,\"status\":\"routed\"}],\"location\":\"Inside motor junction box; M1.PE is the shared three-port interface\"}"
 			(at 245 638 0)
 			(layer "F.Fab")
@@
 	)
 	(segment
-		(start 240 905)
-		(end 240 854)
-		(width 2.588)
-		(layer "In3.Cu")
-		(net "PE")
-	)
-	(segment
 		(start 303 905)
 		(end 240 905)
@@
 	)
 	(segment
-		(start 245 849)
-		(end 263 849)
-		(width 2.588)
-		(layer "In3.Cu")
-		(net "PE")
-	)
-	(segment
 		(start 308 875)
 		(end 308 900)
@@
 		(net "PE")
 	)
-	(arc
-		(start 240 854)
-		(mid 241 851)
-		(end 245 849)
-		(width 2.588)
-		(layer "In3.Cu")
-		(net "PE")
-	)
 	(segment
 		(start 78 205)
@@
 	(footprint "Controls:Frame_PE_Lug_20mm"
 		(layer "F.Cu")
-		(at 450 430)
+		(at 449.2876 449.2876)
 		(descr "PCB-only frame protective-earth lug routing target. User-defined 20 mm circular marker with centered PE THT pad. Logical machine-frame wiring representation; the 3 mm pad and 2 mm drill are routing-target geometry, not installed lug or fastener dimensions.")
 		(tags "frame PE protective earth bonding lug PCB-only")
@@
 			(at 0 12 0)
 			(layer "F.Fab")
+			(hide yes)
 			(effects
 				(font
@@
 			)
 		)
-		(property "Description" "Lower-right manufacturer-provided backplate/enclosure grounding stud, owner-confirmed 5/16 in. Routing target at (450,430) mm rounds saved mounting center (449.5286,430.4786) mm to the 1 mm routing grid. Marker geometry is not hardware or a drilling specification."
+		(property "Description" "Electrical routing endpoint concentric with the existing lower-right grounding fixture in EN4SD30208GY_Open_Front on User.Drawings at (449.2876,449.2876) mm. Reuses enclosure-supplied lug; no new lug or drilling geometry."
 			(at 0 0 0)
 			(layer "F.Fab")
@@
 			)
 		)
-		(property "BOM.CountedIn" "Enclosure-provided grounding stud and mounting hardware. McMaster 9388K35 ring terminal is a separate BOM consumable."
+		(property "BOM.CountedIn" "Enclosure-supplied grounding lug and hardware. McMaster 9388K35 ring terminal is a separate BOM consumable."
 			(at 0 0 0)
 			(layer "F.Fab")
@@
 			)
 		)
-		(property "Wire.BondingPlan" "TB50.1 to J8.PE lower-right enclosure/backplate grounding stud: 12 AWG green/yellow, 10 mm single ferrule at TB50.1 and McMaster 9388K35 5/16 in ring at J8. Routed; retain the four backplate mounting/bonding interfaces."
+		(property "Wire.BondingPlan" "TB50.1 to J8.PE: 12 AWG green/yellow to the existing lower-right enclosure grounding fixture on User.Drawings; endpoint concentric at (449.2876,449.2876) mm. 10 mm single ferrule at TB50.1; owner-selected 5/16 in McMaster 9388K35 ring at the lug."
 			(at 0 0 0)
 			(layer "F.Fab")
@@
 		(attr board_only exclude_from_pos_files exclude_from_bom allow_missing_courtyard)
 		(duplicate_pad_numbers_are_jumpers no)
-		(fp_circle
-			(center 0 0)
-			(end 9 0)
-			(stroke
-				(width 0.2)
-				(type default)
-			)
-			(fill no)
-			(layer "F.SilkS")
-		)
-		(fp_circle
-			(center 0 0)
-			(end 10 0)
-			(stroke
-				(width 0.25)
-				(type default)
-			)
-			(fill no)
-			(layer "F.SilkS")
-		)
-		(fp_circle
-			(center 0 0)
-			(end 10 0)
-			(stroke
-				(width 0.1)
-				(type default)
-			)
-			(fill no)
-			(layer "F.Fab")
-		)
 		(pad "PE" thru_hole circle
 			(at 0 0)
@@
 	)
 	(segment
-		(start 443 210)
-		(end 443 425)
+		(start 243 287)
+		(end 243 210)
 		(width 2.052)
 		(layer "F.Cu")
@@
 	)
 	(segment
-		(start 243 287)
-		(end 243 210)
+		(start 263 849)
+		(end 303 849)
+		(width 2.588)
+		(layer "F.Cu")
+		(net "PE")
+	)
+	(segment
+		(start 248 205)
+		(end 438 205)
 		(width 2.052)
 		(layer "F.Cu")
@@
 	)
 	(segment
-		(start 448 430)
-		(end 450 430)
+		(start 308 854)
+		(end 308 875)
+		(width 2.588)
+		(layer "F.Cu")
+		(net "PE")
+	)
+	(segment
+		(start 443 210)
+		(end 443 444.2876)
 		(width 2.052)
 		(layer "F.Cu")
@@
 	)
 	(segment
-		(start 248 205)
-		(end 438 205)
+		(start 448 449.2876)
+		(end 449.2876 449.2876)
+		(width 2.052)
+		(layer "F.Cu")
+		(net "PE")
+	)
+	(arc
+		(start 438 205)
+		(mid 441.535534 206.464466)
+		(end 443 210)
 		(width 2.052)
 		(layer "F.Cu")
@@
 	)
 	(arc
-		(start 443 425)
-		(mid 444.464466 428.535534)
-		(end 448 430)
-		(width 2.052)
+		(start 303 849)
+		(mid 306.535534 850.464466)
+		(end 308 854)
+		(width 2.588)
 		(layer "F.Cu")
 		(net "PE")
 	)
 	(arc
-		(start 438 205)
-		(mid 441.535534 206.464466)
-		(end 443 210)
+		(start 443 444.2876)
+		(mid 444.464466 447.823134)
+		(end 448 449.2876)
 		(width 2.052)
 		(layer "F.Cu")
